Commit message: Update ROS2 control and MoveIt configs for Fetch robot

File: controllers/fetch_controller/src/fetch_description/config/fetch.ros2_control.xacro (robot description, xacro)
@@ -64,4 +64,11 @@
                 <state_interface name="velocity"/>
             </joint>
+            <joint name="l_gripper_finger_joint">
+                <command_interface name="position"/>
+                <state_interface name="position">
+                  <param name="initial_value">${initial_positions['l_gripper_finger_joint']}</param>
+                </state_interface>
+                <state_interface name="velocity"/>
+            </joint>
             <joint name="r_gripper_finger_joint">
                 <command_interface name="position"/>
