Commit message: Modify fetch.urdf for gripper and sensor updates
Updated inertia properties for gripper fingers and added new links and joints for lidar and camera components.

File: protos/fetch_description/robots/fetch.urdf (robot description, URDF)
Before this commit: robot fetch, 26 links, 25 joints
Links:
- added link camera_link, mass 0.001
- added link depth_camera_link, mass 0.001
- added link lidar1_link, mass 0.001
- added link lidar2_link, mass 0.001
Joints:
- added joint camera_joint: type fixed, parent head_pan_link, child camera_link, origin xyz=0 0 0.1 rpy=0 0 0
- added joint depth_camera_joint: type fixed, parent head_pan_link, child depth_camera_link, origin xyz=0 0 0.1 rpy=0 0 0
- added joint lidar1_joint: type fixed, parent torso_fixed_link, child lidar1_link, origin xyz=0 0 0.2 rpy=0 0 0
- added joint lidar2_joint: type fixed, parent torso_fixed_link, child lidar2_link, origin xyz=0 0 0.2 rpy=0 0 0
